File: hardware/esp-crimpdeq-board/power_management.kicad_sch (KiCad schematic)
At the start: 44 parts, among them J1 USB4105-GF-A, Q1 DMG3415U, U3 REF35330QDBVR, U4 SY8088, U5 SY8088, U6 MCP73831T-2ACI/OT, U7 MAX17262

Commit message: feat: Organice schematic
Other:
- note added: "Battery Gauge"
Changed lines of the file:
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@@
 	(generator_version "9.0")
 	(paper "A4")
+	(rectangle
+		(start 110.49 95.25)
+		(end 198.12 143.51)
+		(stroke
+			(width 0)
+			(type dash)
+		)
+		(fill
+			(type none)
+		)
+	)
 	(text "DC/DC Buck Converter 3V3 Rails"
 		(exclude_from_sim no)
@@
 		(effects
 			(font
+				(size 1.27 1.27)
+				(thickness 0.254)
+				(bold yes)
+			)
+			(justify left bottom)
+		)
+	)
+	(text "Battery Gauge\n"
+		(exclude_from_sim no)
+		(at 112.268 141.224 0)
+		(effects
+			(font
